File: ozinverterkicad.kicad_pcb (KiCad board)
At the start: 2 copper layers, 100 x 100 mm, 69 parts, among them P1 pwrbrd, P2 onled, P3 on/off, P4 temp, P5 ct sense, P6 Active mains, P7 neutral mains, P8 systemled, Q2 tip35c, T1 12vac transforme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

Commit message: added extra ct routed
Parts:
- removed REF** (x4): 1pin, Connect:1pin
- removed currentlimit: 2k, Discret:RV2X4
- added C24: 1n, Capacitors_ThroughHole:C_Disc_D3_P2.5, F.Cu at (151.9, 107.2)
- added C25: 0.1uf, Capacitors_ThroughHole:C_Radial_D5_L6_P2.5, F.Cu at (148.1, 55.6)
- added D1: D, Diodes_ThroughHole:Diode_DO-41_SOD81_Vertical_AnodeUp, F.Cu at (136.9, 120.4)
- added D15: 6v0, Diodes_ThroughHole:Diode_DO-41_SOD81_Vertical_AnodeUp, F.Cu at (148.8, 122.4)
- added D16: oc-fast, LEDs:LED-5MM, F.Cu at (166.6, 71.4)
- added D17: D, Diodes_ThroughHole:Diode_DO-41_SOD81_Vertical_AnodeUp, F.Cu at (157.0, 63.0)
- added D18: D, Diodes_ThroughHole:Diode_DO-41_SOD81_Vertical_AnodeUp, F.Cu at (160.5, 59.7)
- added D19: D, Diodes_ThroughHole:Diode_DO-41_SOD81_Vertical_AnodeUp, F.Cu at (160.5, 56.9)
- added D20: D, Diodes_ThroughHole:Diode_DO-41_SOD81_Vertical_AnodeUp, F.Cu at (157.0, 53.8)
- added JP1: reset, Connectors_Molex:Molex_KK-6410-02_02x2.54mm_Straight, F.Cu at (167.6, 56.6)
- added R1: 10k, Resistors_ThroughHole:Resistor_Horizontal_RM7mm, F.Cu at (122.9, 112.5)
- added R15: 1k, Resistors_ThroughHole:Resistor_Horizontal_RM7mm, F.Cu at (147.6, 102.1)
- added R16: 1k, Resistors_ThroughHole:Resistor_Horizontal_RM7mm, F.Cu at (165.6, 85.3)
- added R17: 1k, Resistors_ThroughHole:Resistor_Horizontal_RM7mm, F.Cu at (153.7, 61.2)
- added R2: 1k8, Resistors_ThroughHole:Resistor_Horizontal_RM7mm, F.Cu at (160.3, 123.2)
- added U5: mcr100, TO_SOT_Packages_THT:TO-92_Molded_Narrow, F.Cu at (158.8, 105.4)
- added ctfast: 2k, Discret:RV2X4, F.Cu at (136.4, 55.9)
- added oc-slow: 2k, Discret:RV2X4, F.Cu at (140.7, 128.5)
- added p1: ct sensefast, Connectors_Molex:Molex_KK-6410-02_02x2.54mm_Straight, F.Cu at (167.4, 64.0)
- P1: value pwrbrd -> CONN_02X05
- P2: value onled -> status
Connections:
- C11 pad 2: Net-(C11-Pad2) -> Net-(C10-Pad2)
- C13 pad 1: Net-(C11-Pad2) -> Net-(C10-Pad2)
- U2 pad 11: Net-(C11-Pad2) -> Net-(C10-Pad2)
Routing:
- net Net-(C24-Pad2): track 20.7 -> 123.8 mm
- net Net-(D15-Pad1): track 0.00 -> 76.9 mm
- net Net-(C24-Pad1): track 0.00 -> 60.3 mm
- net Net-(JP1-Pad2): track 0.00 -> 53.4 mm
- net Net-(C10-Pad2): track 37.9 -> 74.1 mm
- net Net-(C11-Pad2): track 21.3 -> 0.00 mm
- net Net-(D17-Pad1): track 0.00 -> 13.0 mm
- net Net-(D19-Pad1): track 0.00 -> 12.7 mm
- net Net-(C25-Pad1): track 0.00 -> 11.5 mm
- net Net-(D17-Pad2): track 0.00 -> 10.4 mm
- net Net-(D16-Pad2): track 0.00 -> 7.82 mm
- net Net-(C6-Pad2): track 44.4 -> 36.9 mm
- net Net-(R8-Pad1): track 54.7 -> 58.3 mm
- net Net-(R15-Pad2): track 0.00 -> 3.13 mm
- net Net-(R10-Pad2): track 13.1 -> 15.9 mm
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