File: ozinverterkicad.sch (KiCad schematic (older format))
At the start: 83 parts, among them P1 CONN_02X05, P2 status, P3 on/off, P4 temp, P5 ct sense, P6 Active mains, P7 neutral mains, P8 systemled, Q2 tip35c, T1 12vac transforme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

Commit message: changed plug around for correct pinout
Parts:
- D14, D16, D5: symbol LED -> LED-RESCUE-ozinverterkicad
- RV1, RV2, voltageout1: symbol POT -> POT-RESCUE-ozinverterkicad
Connections:
- net +12V: now also U4.2 (GND); no longer U4.1 (PWR_OUt)
- net +48V: now also P1.1 (P1), P1.2 (P2), U4.3 (GND); no longer P1.10 (P10), P1.9 (P9), U4.4 (Pwr_In)
- net GND: now also P1.10 (P10), P1.9 (P9), U4.1 (PWR_OUt), U4.4 (Pwr_In); no longer P1.1 (P1), P1.2 (P2), U4.2 (GND), U4.3 (GND)
- net at P1.3 (P3): now also U1.7 (ho); no longer U1.1 (LO)
- net at P1.7 (P7): now also U1.1 (LO); no longer U1.7 (ho)
Changed lines of the file:
@@
 EESchema Schematic File Version 2
+LIBS:ozinverterkicad-rescue
 LIBS:power
 LIBS:device
@@
 $EndComp
 $Comp
-L LED D5
+L LED-RESCUE-ozinverterkicad D5
 U 1 1 57CA8B3C
 P 5725 4575
@@
 $EndComp
 $Comp
-L POT voltageout1
+L POT-RESCUE-ozinverterkicad voltageout1
 U 1 1 57CA98D3
 P 7450 4175
@@
 $EndComp
 $Comp
-L POT RV1
+L POT-RESCUE-ozinverterkicad RV1
 U 1 1 57CAB4A0
 P 7000 2775
@@
 L GND #PWR019
 U 1 1 57CB3A5E
-P 1500 7400
-F 0 "#PWR019" H 1500 7150 50  0001 C CNN
-F 1 "GND" H 1500 7250 50  0000 C CNN
-F 2 "" H 1500 7400 50  0000 C CNN
-F 3 "" H 1500 7400 50  0000 C CNN
-	1    1500 7400
+P 1100 6450
+F 0 "#PWR019" H 1100 6200 50  0001 C CNN
+F 1 "GND" H 1100 6300 50  0000 C CNN
+F 2 "" H 1100 6450 50  0000 C CNN
+F 3 "" H 1100 6450 50  0000 C CNN
+	1    1100 6450
 	1    0    0    -1
 $EndComp
@@
 L +48V #PWR020
 U 1 1 57CB3D96
-P 1375 6550
-F 0 "#PWR020" H 1375 6400 50  0001 C CNN
-F 1 "+48V" H 1375 6690 50  0000 C CNN
-F 2 "" H 1375 6550 50  0000 C CNN
-F 3 "" H 1375 6550 50  0000 C CNN
-	1    1375 6550
+P 1825 7525
+F 0 "#PWR020" H 1825 7375 50  0001 C CNN
+F 1 "+48V" H 1825 7665 50  0000 C CNN
+F 2 "" H 1825 7525 50  0000 C CNN
+F 3 "" H 1825 7525 50  0000 C CNN
+	1    1825 7525
 	1    0    0    -1
 $EndComp
@@
 $EndComp
 $Comp
-L LED D14
+L LED-RESCUE-ozinverterkicad D14
 U 1 1 57CC6041
 P 4725 1500
@@
 L GND #PWR030
 U 1 1 57CBDA8B
-P 825 1025
-F 0 "#PWR030" H 825 775 50  0001 C CNN
-F 1 "GND" H 825 875 50  0000 C CNN
-F 2 "" H 825 1025 50  0000 C CNN
-F 3 "" H 825 1025 50  0000 C CNN
-	1    825  1025
+P 750 1450
+F 0 "#PWR030" H 750 1200 50  0001 C CNN
+F 1 "GND" H 750 1300 50  0000 C CNN
+F 2 "" H 750 1450 50  0000 C CNN
+F 3 "" H 750 1450 50  0000 C CNN
+	1    750  1450
 	1    0    0    -1
 $EndComp
@@
 L GND #PWR031
 U 1 1 57CBE302
-P 2450 1050
-F 0 "#PWR031" H 2450 800 50  0001 C CNN
-F 1 "GND" H 2450 900 50  0000 C CNN
-F 2 "" H 2450 1050 50  0000 C CNN
-F 3 "" H 2450 1050 50  0000 C CNN
-	1    2450 1050
+P 2325 1150
+F 0 "#PWR031" H 2325 900 50  0001 C CNN
+F 1 "GND" H 2325 1000 50  0000 C CNN
+F 2 "" H 2325 1150 50  0000 C CNN
+F 3 "" H 2325 1150 50  0000 C CNN
+	1    2325 1150
 	1    0    0    -1
 $EndComp
@@
 	1675 6625 1675 6850
 Wire Wire Line
-	1375 6550 1375 6625
+	1375 6450 1375 6625
 Connection ~ 1375 6625
 Wire Wire Line
@@
 	850  6300 1875 6300
 Wire Wire Line
-	1875 6300 1875 7150
-Wire Wire Line
-	1875 7150 1675 7150
+	1875 6300 1875 6950
+Wire Wire Line
+	1975 7150 1675 7150
 Wire Wire Line
 	1700 4600 950  4600
@@
 	950  6200 1925 6200
 Wire Wire Line
-	1925 6200 1925 7050
-Wire Wire Line
 	1925 7050 1675 7050
 Wire Wire Line
@@
 	1050 6150 1975 6150
 Wire Wire Line
-	1975 6150 1975 6950
-Wire Wire Line
-	1975 6950 1675 6950
+	1975 6150 1975 7150
+Wire Wire Line
+	1875 6950 1675 6950
 Wire Wire Line
 	4150 4175 4150 3475
@@
 	5075 1350 5075 1025
 Wire Wire Line
-	650  875  650  1400
-Wire Wire Line
-	650  1400 850  1400
-Wire Wire Line
-	825  1025 850  1025
+	650  1025 850  1025
 Wire Wire Line
 	850  1025 850  1000
@@
 	2450 1000 2450 1050
 Wire Wire Line
-	2450 1400 2750 1400
+	2525 1400 2750 1400
 Wire Wire Line
 	2750 1400 2750 900
@@
 	2275 1550 2525 1550
 Wire Wire Line
-	2525 1550 2525 1400
+	2525 1550 2525 1050
 Connection ~ 2525 1400
 Wire Wire Line
-	7200 1375 7200 1300
+	7200 1300 7200 1375
 Wire Wire Line
 	7200 925  7200 1000
@@
 $EndComp
 $Comp
-L POT RV2
+L POT-RESCUE-ozinverterkicad RV2
 U 1 1 58026D0E
 P 8750 1325
@@
 $EndComp
 $Comp
-L LED D16
+L LED-RESCUE-ozinverterkicad D16
 U 1 1 5802A3B1
 P 8975 2775
@@
 Wire Wire Line
 	2725 5150 2725 5200
+Connection ~ 1875 7150
+Connection ~ 1975 6950
+Connection ~ 1875 6950
+Wire Wire Line
+	1925 6200 1925 7050
+Wire Wire Line
+	650  875  650  1025
+Wire Wire Line
+	750  1450 750  1400
+Wire Wire Line
+	750  1400 850  1400
+Wire Wire Line
+	2450 1400 2450 1150
+Wire Wire Line
+	2450 1150 2325 1150
+Wire Wire Line
+	2525 1050 2450 1050
+Wire Wire Line
+	1100 6450 1375 6450
+Wire Wire Line
+	1500 7400 1500 7525
+Wire Wire Line
+	1500 7525 1825 7525
+Connection ~ 1500 7400
 $EndSCHEMATC
